File: STM32F103C8T6.kicad_pcb (KiCad board)
At the start: 4 copper layers, 65 x 30 mm, 39 parts, among them J3 Conn_01x04, J4 Conn_01x20, J5 Conn_01x20, Y1 32.768kHz, Y2 8MHz

Commit message: Add silk screen,changed some cap
Parts:
- moved R3 2.00 mm to (69.2, 42.8)
- moved C9 1.15 mm to (73.7, 42.8)
- renumbered BOOT to BOOT0
Routing:
- net NRST: track 94.8 -> 84.5 mm
- net GND: track 65.0 -> 59.6 mm, vias 14 -> 15
- net VCC: track 54.6 -> 54.1 mm
Other:
- board text added: "0"
- board text added: "1"
- board text added: "BOOT1"
- board text added: "CLK"
- board text added: "SWD"
